Commit message: fix lidar-imu extrinsics

File: config/robot.urdf.xacro (robot description, xacro)
@@ -11,5 +11,5 @@
   <link name="lidar_link"> </link>
   <joint name="lidar_joint" type="fixed">
-    <parent link="base_link" />
+    <parent link="chassis_link" />
     <child link="lidar_link" />
     <origin xyz="0 0 0" rpy="0 0 0" />

Commit message: rebase Simple-LIO-SAM ros2 && add Hesai Lidar adaptation

File: config/robot.urdf.xacro (robot description, xacro)
@@ -2,32 +2,26 @@
 <robot name="lio" xmlns:xacro="http://tixiaoshan.github.io/">
   <xacro:property name="PI" value="3.1415926535897931" />
-  <link name="chassis_link"></link>
+  <link name="map"></link>
+  <link name="odom"></link>
+  <joint name="map_joint" type="fixed">
+    <origin xyz="0.0 0.0 0.0" rpy="0.0 0.0 0.0"/>
+    <parent link="map"/>
+    <child link="odom"/>
+  </joint>
   <link name="base_link"></link>
-  <joint name="base_link_joint" type="fixed">
-    <parent link="base_link"/>
-    <child link="chassis_link" />
-    <origin xyz="0 0 0" rpy="0 0 0" />
-  </joint>
-  <link name="lidar_link"> </link>
-  <joint name="lidar_joint" type="fixed">
-    <parent link="chassis_link" />
-    <child link="lidar_link" />
-    <origin xyz="0 0 0" rpy="0 0 0" />
+  <joint name="odom_joint" type="continuous">
+    <origin xyz="0.0 0.0 0.0" rpy="0.0 0.0 0.0"/>
+    <parent link="odom"/>
+    <child link="base_link"/>
   </joint>
   <link name="imu_link"> </link>
   <joint name="imu_joint" type="fixed">
-    <parent link="chassis_link" />
+    <parent link="base_link" />
     <child link="imu_link" />
-    <origin xyz="0 0 0" rpy="0 0 0" />
-  </joint>
-  <link name="laser_sensor_frame"> </link>
-  <joint name="laser_joint" type="fixed">
-    <parent link="imu_link" />
-    <child link="laser_sensor_frame" />
     <origin xyz="0 0 0" rpy="0 0 0" />
   </joint>
   <link name="navsat_link"> </link>
   <joint name="navsat_joint" type="fixed">
-    <parent link="chassis_link" />
+    <parent link="base_link" />
     <child link="navsat_link" />
     <origin xyz="0 0 0" rpy="0 0 0" />
